Commit message: david_description / david_moveit_config / david_sdk_bridge: arm home-pose + TCP rework
- david_description: replace hand_base_link with left_arm_fixed_link and
  right_arm_fixed_link meshes; large URDF restructure in
  david_description/urdf/david.urdf. david_nav/urdf/david.urdf trimmed to
  the leaner shared layout.
- david_moveit_config: SRDF tip_link switched from the AR5 flan_link to
  left_tcp / right_tcp; home group_state updated to the new joint_1 values
  (left 1.9199 -> 2.5307, right -1.9199 -> -2.6181); collision-disable
  entries added for the new fixed_link bodies. real_robot.launch.py wraps
  jsp / move_group / rviz in a 3s TimerAction so sdk_bridge can publish
  /joint_states_arms first (otherwise MoveIt boots without arm joints).
- david_sdk_bridge: arm_node declares a home_pose_deg parameter (deg, SDK
  coords) and publishes that pose whenever dry_run is on or the SDK is not
  connected, so RViz always shows the real starting posture. sdk_bridge.
  launch.py sets the SRDF-matching home for left and right arms.
- nav2_go2_view.rviz: TF panel now exposes base_footprint and chassis_root
  and drops the pruned camera frames.

Co-Authored-By: Claude Opus 4.7 (1M context) <noreply@anthropic.com>

File: david_description/urdf/david.urdf (robot description, URDF)
Before this commit: robot waist_robot, 72 links, 71 joints
Links:
- added link left_arm_fixed_link, mass 0.664016072331186; collision mesh filename=package://david_description/meshes/left_arm_fixed_link.STL; visual mesh filename=package://david_description/meshes/left_arm_fixed_link.STL
- added link left_tcp
- added link right_arm_fixed_link, mass 0.664016076750115; collision mesh filename=package://david_description/meshes/right_arm_fixed_link.STL; visual mesh filename=package://david_description/meshes/right_arm_fixed_link.STL
- added link right_tcp
- link Link3: mass 0.760517445677976 -> 0.760517445677975
- link Link4: mass 3.27516013736829 -> 8.73520467499097
- link base_link: mass None -> 22.4651142385164
- link imu_link: mass 0 -> 0.0260716042797142
- link left_hand_base_link: geometry collision mesh filename=package://david_description/meshes/left_hand/hand_base_link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; visual mesh filename=package://david_description/meshes/left_hand/hand_base_link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
- link left_wheel_link: mass 0.27239 -> 0.272387982807766
- link lidar_link: mass 0.9232 -> 0.92319700040443
- link right_wheel_link: mass 0.27239 -> 0.272387983874311
Joints:
- added joint left_arm_fixed_joint: type fixed, parent Link4, child left_arm_fixed_link, origin xyz=0 0.1325 0.276 rpy=0 0 0, axis 0 0 0
- added joint left_tcp_joint: type fixed, parent AR5-5_08L-W4C4A6-ZY2_flan_link, child left_tcp, origin xyz=0 0 0.22 rpy=0 0 0
- added joint right_arm_fixed_joint: type fixed, parent Link4, child right_arm_fixed_link, origin xyz=0 -0.1325 0.276 rpy=0 0 0, axis 0 0 0
- added joint right_tcp_joint: type fixed, parent AR5-5_08R-W4C4A6-ZY2_flan_link, child right_tcp, origin xyz=0 0 0.22 rpy=0 0 0
- joint Joint1: limit lower=0 upper=1.5707 effort=0 velocity=0 -> lower=0 upper=1.5707 effort=10 velocity=3; origin xyz=0.158960837882583 0.188016398930589 0.335999999999998 rpy=0 0 0 -> xyz=0.15896 0.18802 0.336 rpy=0 0 0
- joint Joint2: limit lower=-3.14159 upper=0 effort=0 velocity=0 -> lower=-3.14159 upper=0 effort=10 velocity=3; origin xyz=-0.395002505835281 -0.0177249999999986 0.0630318997321883 rpy=0 0 0 -> xyz=-0.395 -0.017725 0.063032 rpy=0 0 0
- joint Joint3: limit lower=-1.57 upper=1.57 effort=0 velocity=0 -> lower=-0.785 upper=0.785 effort=10 velocity=3; origin xyz=0.320000000000001 -0.0237250000000076 0.05901429787681 rpy=0 0 0 -> xyz=0.32 -0.023725 0.059014 rpy=0 0 0
- joint Joint4: origin xyz=0 -0.147675 0.167499999998591 rpy=0 0 0 -> xyz=0 -0.14768 0.1675 rpy=0 0 0
- joint index_pip: mimic (none) -> joint=index_mcp_pitch multiplier=1.0 offset=0
- joint left_arm_connect: origin xyz=0 0.1047 0.276 rpy=-1.570 0 0 -> xyz=0 0 0 rpy=-1.570 0 0; parent Link4 -> left_arm_fixed_link
- joint left_index_pip: mimic (none) -> joint=left_index_mcp_pitch multiplier=1.0 offset=0
- joint left_middle_pip: mimic (none) -> joint=left_middle_mcp_pitch multiplier=1.0 offset=0
- joint left_pinky_pip: mimic (none) -> joint=left_pinky_mcp_pitch multiplier=1.0 offset=0
- joint left_ring_pip: mimic (none) -> joint=left_ring_mcp_pitch multiplier=1.0 offset=0
- joint left_thumb_mcp: mimic (none) -> joint=left_thumb_cmc_pitch multiplier=1.33 offset=0
- joint middle_pip: mimic (none) -> joint=middle_mcp_pitch multiplier=1.0 offset=0
- joint pinky_pip: mimic (none) -> joint=pinky_mcp_pitch multiplier=1.0 offset=0
- joint right_arm_connect: origin xyz=0 -0.1047 0.276 rpy=1.570 0 0 -> xyz=0 0 0 rpy=1.570 0 0; parent Link4 -> right_arm_fixed_link
- joint ring_pip: mimic (none) -> joint=ring_mcp_pitch multiplier=1.0 offset=0
- joint thumb_mcp: mimic (none) -> joint=thumb_cmc_pitch multiplier=1.33 offset=0
