Commit message: 机械臂抓取任务 5.19: Stage 0 TCP frame + waist 规划组 + Stage 1 灵巧手 ROS 集成
- david_description: 迁移厂家新版 URDF; 末尾加 left_tcp/right_tcp frame (z=0.22m on flan_link)
- david_moveit_config: left_arm/right_arm tip_link 改为 TCP; 新增 waist 规划组 (base_link->Link4, Joint1-4);
  home group_state 同步真机实测姿态; real_robot.launch.py 延迟 3s 启动避免 RViz T-pose;
  mock_components 给 Joint1-4 设 initial_value
- david_sdk_bridge: arm_node 集成 L10HandController (share robot, 不重复 connect);
  连不上真机自动 fallback 到 mock 模式; 新增灵巧手 service /{side}_hand/set_pose10 + /preset,
  topic /{side}_hand/state (2Hz pose+effort+vel, 3帧中位数滤波); sdk_bridge.launch.py 加 hand_slave_id
- david_hand_msgs: 新建接口定义包 (SetHandPose.srv / SetHandPreset.srv)
- david_grasp: 新建视觉抓取仓库骨架 (Stage 3-5 代码归集位置)

File: david_description/urdf/david.urdf (robot description, URDF)
Before this commit: robot waist_robot, 76 links, 75 joints
Joints:
- joint index_pip: mimic joint=index_mcp_pitch multiplier=1.0 offset=0 -> joint=index_mcp_pitch multiplier=1 offset=0
- joint left_arm_connect: origin xyz=0 0 0 rpy=-1.570 0 0 -> xyz=0 -0.09 0 rpy=-1.570 0 0
- joint left_index_pip: mimic joint=left_index_mcp_pitch multiplier=1.0 offset=0 -> joint=left_index_mcp_pitch multiplier=1 offset=0
- joint left_middle_pip: mimic joint=left_middle_mcp_pitch multiplier=1.0 offset=0 -> joint=left_middle_mcp_pitch multiplier=1 offset=0
- joint left_pinky_pip: mimic joint=left_pinky_mcp_pitch multiplier=1.0 offset=0 -> joint=left_pinky_mcp_pitch multiplier=1 offset=0
- joint left_ring_pip: mimic joint=left_ring_mcp_pitch multiplier=1.0 offset=0 -> joint=left_ring_mcp_pitch multiplier=1 offset=0
- joint left_thumb_mcp: mimic joint=left_thumb_cmc_pitch multiplier=1.33 offset=0 -> (none)
- joint middle_pip: mimic joint=middle_mcp_pitch multiplier=1.0 offset=0 -> joint=middle_mcp_pitch multiplier=1 offset=0
- joint pinky_pip: mimic joint=pinky_mcp_pitch multiplier=1.0 offset=0 -> joint=pinky_mcp_pitch multiplier=1 offset=0
- joint right_arm_connect: origin xyz=0 0 0 rpy=1.570 0 0 -> xyz=0 0.09 0 rpy=1.570 0 0
- joint ring_pip: mimic joint=ring_mcp_pitch multiplier=1.0 offset=0 -> joint=ring_mcp_pitch multiplier=1 offset=0
- joint thumb_mcp: mimic joint=thumb_cmc_pitch multiplier=1.33 offset=0 -> (none)

File: david_moveit_config/config/david.urdf.xacro (robot description, xacro)
@@ -9,6 +9,6 @@
       <command_interface name="position"/>
       <state_interface name="position">
-        <param name="initial_value">0.0</param>
-      </state_interface>
+          <param name="initial_value">0.3316</param>
+        </state_interface>
       <state_interface name="velocity"/>
     </joint>
@@ -16,6 +16,6 @@
       <command_interface name="position"/>
       <state_interface name="position">
-        <param name="initial_value">0.0</param>
-      </state_interface>
+          <param name="initial_value">-0.5934</param>
+        </state_interface>
       <state_interface name="velocity"/>
     </joint>
@@ -23,6 +23,6 @@
       <command_interface name="position"/>
       <state_interface name="position">
-        <param name="initial_value">0.0</param>
-      </state_interface>
+          <param name="initial_value">0.2618</param>
+        </state_interface>
       <state_interface name="velocity"/>
     </joint>
@@ -30,6 +30,6 @@
       <command_interface name="position"/>
       <state_interface name="position">
-        <param name="initial_value">0.0</param>
-      </state_interface>
+          <param name="initial_value">0.0000</param>
+        </state_interface>
       <state_interface name="velocity"/>
     </joint>

Commit message: david_grasp + arm_node: vision-driven bottle grasp (milestone 1)
- new david_grasp/pick_from_cam.py: end-to-end vision -> tf2 -> ikpy IK -> MoveIt -> L10 grasp
  - subscribes /grasp/right/detection (B YOLO+RealSense JSON), only P_cam used
  - tf2 via OUR URDF camera_link (not B handeye yaml; verified 3-axis <1.5cm)
  - 3-tier IK fallback (full / z_only / position) + dual-axis orientation filter
  - modes: hover / approach / grasp (= open hand -> move -> close -> lift)
  - custom OPEN_HAND_POSE [255,0,255,255,255,255,128,128,128,128] thumb_yaw=0

- new david_grasp/goto_pose.py: standalone arm goto by xyz (no vision)
- new david_grasp/set_hand_pose.py: one-shot 10-vec hand pose setter
- new david_grasp/mock_grasp_pose.py: stand-in publisher for offline testing
- new david_grasp/pick_cartesian.py: earlier PoseStamped variant kept for ref
- new david_grasp/greet.py

- david_description/urdf/david.urdf: add camera_link under Link4 (xyz 0.09 0 0.535, pitch 0.838 rad ~48deg)
- david_sdk_bridge/arm_node.py: init hand torque=150 speed=120 at boot (fixes right hand not moving)
- david_sdk_bridge/arm_node.py: race-fix prelude before idle-poll; trajectory simplify to goal-only
- david_moveit_config/kinematics.yaml: KDL timeout 0.05->0.5, attempts 3->100
- david_moveit_config/moveit_controllers.yaml: allowed_execution_duration_scaling 5.0

Milestone 1 achieved 2026-05-29 (one day early); ~80% success rate over 20+ multi-position trials.

File: david_description/urdf/david.urdf (robot description, URDF)
Before this commit: robot waist_robot, 76 links, 75 joints
Links:
- added link camera_link
Joints:
- added joint link4_to_camera_link: type fixed, parent Link4, child camera_link, origin xyz=0.09 0 0.535 rpy=0 0.838 0

Commit message: feat: 左手 vision grasp 跑通 + AI 组 WS 联调全链路 + estop logging + URDF TF 修复
主要工作 (2026-06-01 ~ 06-03):

【左手 vision grasp 跑通 (6.2 里程碑)】
- pick_from_cam.py: side-aware 重构 + tcp_offset (0.06, 0.04, 0.13) /
  lift_offset (0.04, -0.06, 0.13) 经验校准
- TIGHT_CLOSE_POSE 五指 pitch=155 取代 preset 'grasp', set_pose10 直发
- workspace 预检 / wrist 约束 / IK 3-tier fallback (full/z_only/position)
- 5/7 真机抓取成功率

【AI 组 WS 联调 (6.2 happy path 通)】
- 新建 arm_grab_ws_client.py (370 行): WebSocket 客户端 +
  MultiThreadedExecutor + 自动重连 + 7 个 atomic tools
  (grab_bottle / grab_object / place_object / cancel /
   get_arm_status / arm_home / handover_water) + 11 个错误码 +
  suggested_action 字段 + holding state 跟踪
- main() 开头 pop 掉 Clash 代理 env 防 LAN 流量被劫持
- grab_server.py: HTTP MVP (后被 WS 客户端取代,保留作参考)
- setup.py: 注册 arm_grab_ws_client / grab_server 入口

【estop / silent dry_run 检测 (6.3)】
- arm_node.py: 新增 _ec_readable / _ec_failed / _safe_power_state /
  _is_estop 4 个辅助方法 (基于 Rokae SDK PyErrorCode + PowerState)
- moveStart 后立刻检查 ec != 0, 拒绝即 abort + log 人话错误码
- wait-loop (pre-move 2s + execution 长 loop) 加 estop 检测, 每 250ms
  查一次 powerState, 检测到 estop 立刻 abort
- 消除 'SDK 返回 SUCCESS 但机械臂没动' 的链路 silent fail

【URDF TF 修复 (6.3)】
- left_arm_connect joint: rpy='1.5707963 0 3.1415927' (Rx+90 + Rz+180)
  → rpy='-1.5707963 0 0' (Rx-90 only)
- 修正 cam_to_arm_base TF 链 X/Y/Z 全反号问题, bottle in arm_base
  现在三正坐标, IK 成功率恢复

【sign-flip 回滚 (6.1 末尾 + 6.2 验证)】
- sdk_bridge.launch.py: 左臂 joint_signs 回到 [1]*7
- pick_at_pose.py: LEFT_POSES 回到 5.26 原值
- 确认 URDF base Rx(±90°) 已天然处理两臂对称, 不需要 motor 层翻转

跳过: david_nav/* 改动 (按 user 要求不动 nav 包)

File: david_description/urdf/david.urdf (robot description, URDF)
Before this commit: robot waist_robot, 77 links, 76 joints
Joints:
- joint left_arm_connect: origin xyz=0 -0.09 0 rpy=-1.570 0 0 -> xyz=0 -0.09 0 rpy=-1.5707963 0 0
- joint left_hand_connect: origin xyz=0 0 0 rpy=0 0 0 -> xyz=0 0 0 rpy=0 0 3.1415927

Commit message: fix(urdf): 自带 D455 optical frames, 根治 TF 依赖外部发布
camera_link -> camera_color_optical_frame (xyz 0 -0.059 0, color 传感器物理偏移)
camera_link -> camera_depth_optical_frame (xyz 0)
rpy 均为 REP-103 body->optical (-pi/2, 0, -pi/2)

背景 (2026-06-10 排查):
- perception 侧 start_yolo.sh 自带 RSP + waist_robot.urdf(left_arm_connect
  仍是 6.2 旧值 Rx+90+Rz180), 双 RSP 打架把我们的 TF 覆盖 -> bottle 坐标
  X/Y 反号 -> IK 全 fail
- 同事 pipeline 还把 realsense publish_tf 关了, optical frame 只活在他们
  RSP 里; 杀掉他们 RSP 后 frame 直接消失
- 本 fix 让我们 launch 自给自足; 配套修复(他们仓库): waist_robot.urdf
  rpy 对齐 + start_yolo.sh pkill 限域 + RSP 复用守卫
验证: arm_base<-optical = [0.090,-0.259,-0.102], 对齐 6.5 known-good 至 1mm

File: david_description/urdf/david.urdf (robot description, URDF)
Before this commit: robot waist_robot, 77 links, 76 joints
Links:
- added link camera_color_optical_frame
- added link camera_depth_optical_frame
Joints:
- added joint camera_link_to_color_optical: type fixed, parent camera_link, child camera_color_optical_frame, origin xyz=0 -0.059 0 rpy=-1.5707963 0 -1.5707963
- added joint camera_link_to_depth_optical: type fixed, parent camera_link, child camera_depth_optical_frame, origin xyz=0 0 0 rpy=-1.5707963 0 -1.5707963

Commit message: 6.10更新

File: david_description/urdf/david.urdf (robot description, URDF)
Before this commit: robot waist_robot, 79 links, 78 joints
Joints:
- removed joint camera_link_to_color_optical
- removed joint camera_link_to_depth_optical
- added joint camera_color: type fixed, parent Link4, child camera_color_optical_frame, origin xyz=0.0936 0.015 0.5112 rpy=0.7330382858376184 3.141592653589793 1.5707963267948966
- added joint camera_depth: type fixed, parent Link4, child camera_depth_optical_frame, origin xyz=0.0936 0 0.5112 rpy=0.7330382858376184 3.141592653589793 1.5707963267948966
- joint left_arm_connect: origin xyz=0 -0.09 0 rpy=-1.5707963 0 0 -> xyz=0 -0.09 0 rpy=1.5707963 0 3.1415927
