Commit message: nav(urdf): 双轮前移16.5cm/轮距50.5cm/轮半径22cm + 旋转中心与footprint随动
- 双轮沿base_link +X前移0.165m,轮距对称50.5cm(left/right_wheel_joint)
- base_footprint(=两轮轴中点=差分旋转中心)随之前移到x=0.165;z由轮半径
  0.22推出真实地面=-0.4075(旧-0.25是旧小轮残留,顺带修正激光滤地基准)
- URDF顶部加"差分几何单一真值源"注释块,3个origin由wheel_x_offset/
  half_track/wheel_z/wheel_radius推导,下次底盘差分更新只改URDF
- nav2_params footprint多边形随base_footprint前移重表达(local+global):
  X[-0.30..0.42]->[-0.465..0.255],inscribed 0.30->0.255(膨胀0.40仍≥)
- 旧URDF备份为.bak.20260622_pre_wheel_fwd;附设计/实施说明文档

影响:TF树/RViz/costmap footprint;base_link/laser/imu本体几何不动

Co-Authored-By: Claude Opus 4.8 <noreply@anthropic.com>

File: david_nav/urdf/david.urdf (robot description, URDF)
Before this commit: robot david, 7 links, 6 joints
Joints:
- joint base_link_to_base_footprint: origin xyz=0 0 -0.25 rpy=0 0 0 -> xyz=0.165 0 -0.4075 rpy=0 0 0
- joint left_wheel_joint: origin xyz=-0.2955 0 -0.084 rpy=1.5708 0 0 -> xyz=-0.2525 0.165 -0.084 rpy=1.5708 0 0
- joint right_wheel_joint: origin xyz=0.2969 0 -0.084 rpy=1.5708 0 0 -> xyz=0.2525 0.165 -0.084 rpy=1.5708 0 0
