Commit message: refactor: establish the single navigation pipeline
Route aliases 20, 24, and 21 through navrun/navcfg/nav.launch and remove the retired david_nav, david_cmd, slam_gt, controller bench, scan bridge, custom costmap, compatibility, and golden-test paths.

This keeps production rollback aliases and localization untouched. It does not constitute live navigation or motion acceptance.

Co-Authored-By: OpenAI Codex <codex@openai.com>

File: david_config/urdf/david.urdf (robot description, URDF)
Before this commit: robot david, 7 links, 6 joints
Links:
- link chassis_root: geometry collision mesh filename=package://david_config/meshes/zongzhuang/base_link.STL; visual mesh filename=package://david_config/meshes/zongzhuang/base_link.STL
- link left_wheel_link: geometry collision mesh filename=package://david_config/meshes/zongzhuang/left_wheel_link.STL; visual mesh filename=package://david_config/meshes/zongzhuang/left_wheel_link.STL
- link right_wheel_link: geometry collision mesh filename=package://david_config/meshes/zongzhuang/right_wheel_link.S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; visual mesh filename=package://david_config/meshes/zongzhuang/right_wheel_link.S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
